File: pcb/speakeasy/speakeasy/Speakeasy.kicad_sch (KiCad schematic)
At the start: 21 parts, among them J1 PH-6P立贴, J2 210-A-SMD/02, SW1 BOOT, SW2 RST, U1 ESP32-S3-MINI-1U-N4R2, U2 MAX98357AETE+T, U3 AMS1117-3.3

Commit message: meh
Parts:
- removed C1, C2, C3: 10uF, Capacitor_SMD:C_0805_2012Metric, symbol Device:C
- removed C4, C6: 100nF, Capacitor_SMD:C_0402_1005Metric, symbol Device:C
- removed C5: 1uF, Capacitor_SMD:C_0402_1005Metric, symbol Device:C
- removed J1: PH-6P立贴, EasyEDA:CONN-SMD_6P-P2.0-L14.0-W5.4, symbol EasyEDA:PH-6P立贴
- removed J2: 210-A-SMD/02, EasyEDA:CONN-SMD_210-A-SMD-02, symbol EasyEDA:210-A-SMD_02
- removed R1, R2: 5.1k, Resistor_SMD:R_0402_1005Metric, symbol Device:R
- removed R3: 10k, Resistor_SMD:R_0402_1005Metric, symbol Device:R
- removed R4: 100k, Resistor_SMD:R_0402_1005Metric, symbol Device:R
- removed SW1: BOOT, Button_Switch_SMD:SW_SPST_CK_RS282G05A3, symbol Switch:SW_Push
- removed SW2: RST, Button_Switch_SMD:SW_SPST_CK_RS282G05A3, symbol Switch:SW_Push
- removed TP1: 3V3, TestPoint:TestPoint_Pad_D1.5mm, symbol Connector:TestPoint
- removed TP2: GND, TestPoint:TestPoint_Pad_D1.5mm, symbol Connector:TestPoint
- removed TP3: TXD0, TestPoint:TestPoint_Pad_D1.5mm, symbol Connector:TestPoint
- removed TP4: RXD0, TestPoint:TestPoint_Pad_D1.5mm, symbol Connector:TestPoint
- removed U1: ESP32-S3-MINI-1U-N4R2, EasyEDA:BULETM-SMD_ESPRESSIF_ESP32-S3-MINI-1U-N8, symbol EasyEDA:ESP32-S3-MINI-1U-N4R2
- removed U2: MAX98357AETE+T, EasyEDA:TQFN-16_L3.0-W3.0-P0.50-BL-EP1.5, symbol EasyEDA:MAX98357AETE+T
- removed U3: AMS1117-3.3, EasyEDA:SOT-223-3_L6.5-W3.4-P2.30-LS7.0-BR, symbol EasyEDA:AMS1117-3.3

Commit message: Revert "meh"
This reverts commit 6076602b22e367b01dca4988bd9ac845172b2725.
Parts:
- added C1, C2, C3: 10uF, Capacitor_SMD:C_0805_2012Metric, symbol Device:C
- added C4, C6: 100nF, Capacitor_SMD:C_0402_1005Metric, symbol Device:C
- added C5: 1uF, Capacitor_SMD:C_0402_1005Metric, symbol Device:C
- added J1: PH-6P立贴, EasyEDA:CONN-SMD_6P-P2.0-L14.0-W5.4, symbol EasyEDA:PH-6P立贴
- added J2: 210-A-SMD/02, EasyEDA:CONN-SMD_210-A-SMD-02, symbol EasyEDA:210-A-SMD_02
- added R1, R2: 5.1k, Resistor_SMD:R_0402_1005Metric, symbol Device:R
- added R3: 10k, Resistor_SMD:R_0402_1005Metric, symbol Device:R
- added R4: 100k, Resistor_SMD:R_0402_1005Metric, symbol Device:R
- added SW1: BOOT, Button_Switch_SMD:SW_SPST_CK_RS282G05A3, symbol Switch:SW_Push
- added SW2: RST, Button_Switch_SMD:SW_SPST_CK_RS282G05A3, symbol Switch:SW_Push
- added TP1: 3V3, TestPoint:TestPoint_Pad_D1.5mm, symbol Connector:TestPoint
- added TP2: GND, TestPoint:TestPoint_Pad_D1.5mm, symbol Connector:TestPoint
- added TP3: TXD0, TestPoint:TestPoint_Pad_D1.5mm, symbol Connector:TestPoint
- added TP4: RXD0, TestPoint:TestPoint_Pad_D1.5mm, symbol Connector:TestPoint
- added U1: ESP32-S3-MINI-1U-N4R2, EasyEDA:BULETM-SMD_ESPRESSIF_ESP32-S3-MINI-1U-N8, symbol EasyEDA:ESP32-S3-MINI-1U-N4R2
- added U2: MAX98357AETE+T, EasyEDA:TQFN-16_L3.0-W3.0-P0.50-BL-EP1.5, symbol EasyEDA:MAX98357AETE+T
- added U3: AMS1117-3.3, EasyEDA:SOT-223-3_L6.5-W3.4-P2.30-LS7.0-BR, symbol EasyEDA:AMS1117-3.3
Connections:
- new net +3.3V: C1.2, C2.1, C3.1, C4.1, C5.2, C6.2, J1.1, J1.4, J1.5, J1.7, J1.8, R1.1, R2.1, R3.1, R4.1, SW1.2, SW2.1, SW2.2, TP1.1, TP2.1, U1.3 (3V3), U1.45 (EN), U1.65 (GND), U2.17 (EP), U2.3 (GND), U2.4 (~{SD_MODE}), U3.1 (GND), U3.2 (VOUT)
- new net +5V: C1.1, C5.1, C6.1, J1.6, U2.7 (VDD), U3.3 (VIN)
- new net GPIO0: SW1.1, U1.4 (IO0)
- new net I2S_BCLK: U1.9 (IO5), U2.16 (BCLK)
- new net I2S_DOUT: U1.8 (IO4), U2.1 (DIN)
- new net I2S_LRCLK: U1.10 (IO6), U2.14 (LRCLK)
- new net SPKR_N: J2.2, U2.10 (OUTN)
- new net SPKR_P: J2.1, U2.9 (OUTP)
- new net UART_RX: TP4.1, U1.40 (RXD0)
- new net UART_TX: TP3.1, U1.39 (TXD0)
- new net USB_DM: J1.3, U1.23 (IO19)
- new net USB_DP: J1.2, U1.24 (IO20)

Commit message: wip
Parts:
- removed C1, C2, C3: 10uF, Capacitor_SMD:C_0805_2012Metric, symbol Device:C
- removed C4, C6: 100nF, Capacitor_SMD:C_0402_1005Metric, symbol Device:C
- removed C5: 1uF, Capacitor_SMD:C_0402_1005Metric, symbol Device:C
- removed R1, R2: 5.1k, Resistor_SMD:R_0402_1005Metric, symbol Device:R
- removed R3: 10k, Resistor_SMD:R_0402_1005Metric, symbol Device:R
- removed R4: 100k, Resistor_SMD:R_0402_1005Metric, symbol Device:R
- removed SW1: BOOT, Button_Switch_SMD:SW_SPST_CK_RS282G05A3, symbol Switch:SW_Push
- removed SW2: RST, Button_Switch_SMD:SW_SPST_CK_RS282G05A3, symbol Switch:SW_Push
- added C1, C2, C3: 10uF, EasyEDA:C0805, symbol EasyEDA:CL21A106KAYNNNE
- added C4, C6, C8: 100nF, EasyEDA:C0603, symbol EasyEDA:CC0603KRX7R9BB104
- added C5, C7: 1uF, EasyEDA:C0402, symbol EasyEDA:CL05A105KA5NQNC
- added J3: 210-A-SMD/02, EasyEDA:CONN-SMD_210-A-SMD-02, symbol EasyEDA:210-A-SMD_02
- added R1, R2: 5.1k, EasyEDA:R0402, symbol EasyEDA:0402WGF5101TCE
- added R3: 10k, EasyEDA:R0402, symbol EasyEDA:0402WGF1002TCE
- added R4, R6: 1k, EasyEDA:R0402, symbol EasyEDA:0402WGF1001TCE
- added R5, R7: 100k, EasyEDA:R0402, symbol EasyEDA:0402WGF1003TCE
- added SW1: BOOT, EasyEDA:SW-SMD_4P-L5.1-W5.1-P3.70-LS6.5-TL_H1.5, symbol EasyEDA:TS-1187A-B-A-B
- added SW2: RST, EasyEDA:SW-SMD_4P-L5.1-W5.1-P3.70-LS6.5-TL_H1.5, symbol EasyEDA:TS-1187A-B-A-B
- added U4: MAX98357AETE+T, EasyEDA:TQFN-16_L3.0-W3.0-P0.50-BL-EP1.5, symbol EasyEDA:MAX98357AETE+T
Connections:
- net +3.3V: now also U3.4 (VOUT), C2.1, C3.1, C4.1, R3.1; no longer J1.1, J1.4, J1.5, J1.7, J1.8, TP2.1, U1.45 (EN), U1.65 (GND), U2.17 (EP), U2.3 (GND), U2.4 (~{SD_MODE}), U3.1 (GND)
- net +5V: now also U2.8 (VDD), C1.1, C5.1, C6.1, C7.1, C8.1, U4.7 (VDD), U4.8 (VDD)
- net GPIO0: now also SW1.1 (A)
- net I2S_BCLK: now also U4.16 (BCLK)
- net I2S_DOUT: now also U4.1 (DIN)
- net I2S_LRCLK: now also U4.14 (LRCLK)
- net GND: now reaches U1.1 (GND)
- net GND: now also J1.1, J1.7, J1.8, TP2.1, U1.2 (GND), U1.42 (GND), U1.43 (GND), U1.46 (GND), U1.47 (GND), U1.48 (GND), U1.49 (GND), U1.50 (GND), U1.51 (GND), U1.52 (GND), U1.53 (GND), U1.54 (GND), U1.55 (GND), U1.56 (GND), U1.57 (GND), U1.58 (GND), U1.59 (GND), U1.60 (GND), U1.61 (GND), U1.62 (GND), U1.63 (GND), U1.64 (GND), U1.65 (GND), U2.11 (GND), U2.15 (GND), U2.17 (EP), U2.3 (GND), U3.1 (GND), C1.2, C2.2, C3.2, C4.2, C5.2, C6.2, C7.2, C8.2, R1.2, R2.2, SW1.3 (C), SW2.3 (C), U4.11 (GND), U4.15 (GND), U4.17 (EP), U4.3 (GND)
- net SD_CTRL_A: now reaches U1.11 (IO7)
- net SD_CTRL_A: now also R4.1
- net SD_CTRL_B: now reaches U1.12 (IO8)
- net SD_CTRL_B: now also R5.1
- net SD_CTRL2_A: now reaches U1.13 (IO9)
- net SD_CTRL2_A: now also R6.1
- net SD_CTRL2_B: now reaches U1.14 (IO10)
- net SD_CTRL2_B: now also R7.1
- new net CC1: J1.5, R1.1
- new net CC2: J1.4, R2.1
- new net EN: R3.2, SW2.1 (A), U1.45 (EN)
- new net SD_MODE: R4.2, R5.2, U2.4 (~{SD_MODE})
- new net SD_MODE2: R6.2, R7.2, U4.4 (~{SD_MODE})
- new net SPKR2_N: J3.2, U4.10 (OUTN)
- new net SPKR2_P: J3.1, U4.9 (OUTP)
Other:
- moved on the sheet: J1, J2, TP1, TP2, TP3, TP4, U3

Commit message: 1ch again
Parts:
- removed C7: 1uF, EasyEDA:C0402, symbol EasyEDA:CL05A105KA5NQNC
- removed C8: 100nF, EasyEDA:C0603, symbol EasyEDA:CC0603KRX7R9BB104
- removed J3: 210-A-SMD/02, EasyEDA:CONN-SMD_210-A-SMD-02, symbol EasyEDA:210-A-SMD_02
- removed R6: 1k, EasyEDA:R0402, symbol EasyEDA:0402WGF1001TCE
- removed R7: 100k, EasyEDA:R0402, symbol EasyEDA:0402WGF1003TCE
- removed U4: MAX98357AETE+T, EasyEDA:TQFN-16_L3.0-W3.0-P0.50-BL-EP1.5, symbol EasyEDA:MAX98357AETE+T
Connections:
- net SD_CTRL2_A: no longer names the net of U1.13 (IO9)
- net SD_CTRL2_B: no longer names the net of U1.14 (IO10)
Other:
- moved on the sheet: C1, C2, C3, C4, C5, C6, J1, J2, R1, R2, R3, R4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
