File: pcb/speakeasy/speakeasy/Speakeasy.kicad_sch (KiCad schematic)
At the start: 22 parts, among them J1 PH-6P立贴, J2 210-A-SMD/02, SW1 BOOT, SW2 RST, U1 ESP32-S3-MINI-1U-N4R2, U2 MAX98357AETE+T, U3 AMS1117-3.3

Commit message: v1
Parts:
- removed C1, C2, C3: 10uF, EasyEDA:C0805, symbol EasyEDA:CL21A106KAYNNNE
- removed C4, C6: 100nF, EasyEDA:C0603, symbol EasyEDA:CC0603KRX7R9BB104
- removed SW1: BOOT, EasyEDA:SW-SMD_4P-L5.1-W5.1-P3.70-LS6.5-TL_H1.5, symbol EasyEDA:TS-1187A-B-A-B
- removed SW2: RST, EasyEDA:SW-SMD_4P-L5.1-W5.1-P3.70-LS6.5-TL_H1.5, symbol EasyEDA:TS-1187A-B-A-B
- removed U3: AMS1117-3.3, EasyEDA:SOT-223-3_L6.5-W3.4-P2.30-LS7.0-BR, symbol EasyEDA:AMS1117-3.3
- added C1: 10uF, EasyEDA:C0603, symbol EasyEDA:CL10A106KP8NNNC
- added C2: 10uF, EasyEDA:C0402, symbol EasyEDA:CL05A106MQ5NUNC
- added C3, C6: 100nF, EasyEDA:C0402, symbol EasyEDA:CL05B104KO5NNNC
- added H1, H2, H3, H4: MountingHole, MountingHole:MountingHole_3.2mm_M3_Pad_Via, symbol Mechanical:MountingHole_Pad
- added SW1: BOOT, EasyEDA:SW-SMD_L3.9-W3.0-P4.45, symbol EasyEDA:TS-1088-AR02016
- added SW2: RST, EasyEDA:SW-SMD_L3.9-W3.0-P4.45, symbol EasyEDA:TS-1088-AR02016
- added U3: MPM3810GQB-33-Z, EasyEDA:QFN-12_L3.0-W2.5_MPM3810AGQB-AEC1, symbol EasyEDA:MPM3810GQB-33-Z
Connections:
- net +3.3V: now also C2.1, C3.1, U3.12 (OUT_S), U3.5 (OUT)
- net +5V: now also C1.1, C6.1, U3.7 (VIN), U3.9 (EN)
- net EN: now also SW2.1
- net GND: now also C1.2, C2.2, C3.2, C6.2, H1.1, H2.1, H3.1, H4.1, SW1.2, SW2.2, U3.1 (PGND), U3.11 (AGND), U3.2 (PGND)
- net GPIO0: now also SW1.1
Other:
- moved on the sheet: C5, J1, J2, R1, R2, R3, R4, R5, TP1, TP2, TP3, TP4
