File: pcb/speakeasy/speakeasy/Speakeasy.kicad_pcb (KiCad board)
At the start: 2 copper layers, 70.5 x 41 mm, 21 parts, among them J1 PH-6P立贴, J2 210-A-SMD/02, SW1 BOOT, SW2 RST, U1 ESP32-S3-MINI-1U-N4R2, U2 MAX98357AETE+T, U3 AMS1117-3.3

Commit message: v1
Parts:
- removed C4: 100nF, Capacitor_SMD:C_0402_1005Metric
- added H1: MountingHole, MountingHole:MountingHole_3.2mm_M3_Pad_Via, F.Cu at (134.0, 84.0)
- added H2: MountingHole, MountingHole:MountingHole_3.2mm_M3_Pad_Via, F.Cu at (166.0, 84.0)
- added H3: MountingHole, MountingHole:MountingHole_3.2mm_M3_Pad_Via, F.Cu at (134.0, 116.0)
- added H4: MountingHole, MountingHole:MountingHole_3.2mm_M3_Pad_Via, F.Cu at (166.0, 116.0)
- added R5: 100k, EasyEDA:R0402, F.Cu at (143.0, 98.2)
- C1: footprint Capacitor_SMD:C_0805_2012Metric -> EasyEDA:C0603
- C2: footprint Capacitor_SMD:C_0805_2012Metric -> EasyEDA:C0402
- C3: value 10uF -> 100nF; footprint Capacitor_SMD:C_0805_2012Metric -> EasyEDA:C0402
- C5, C6: footprint Capacitor_SMD:C_0402_1005Metric -> EasyEDA:C0402
- R1, R2, R3: footprint Resistor_SMD:R_0402_1005Metric -> EasyEDA:R0402
- R4: value 100k -> 1k; footprint Resistor_SMD:R_0402_1005Metric -> EasyEDA:R0402
- SW1, SW2: footprint Button_Switch_SMD:SW_SPST_CK_RS282G05A3 -> EasyEDA:SW-SMD_L3.9-W3.0-P4.45; moved to F.Cu
- U3: value AMS1117-3.3 -> MPM3810GQB-33-Z; footprint EasyEDA:SOT-223-3_L6.5-W3.4-P2.30-LS7.0-BR -> EasyEDA:QFN-12_L3.0-W2.5_MPM3810AGQB-AEC1
- moved SW1 82.7 mm to (163.0, 105.5), turned to 0 degrees
- moved C1 77.7 mm to (163.0, 109.2), turned to -90 degrees
- moved C2 74.7 mm to (159.8, 112.2), turned to -90 degrees
- moved C3 72.2 mm to (158.5, 112.2), turned to -90 degrees
- moved TP1 62.9 mm to (155.6, 117.5), turned to 90 degrees
- moved SW2 60.8 mm to (139.2, 110.0)
- moved R3 59.8 mm to (141.2, 113.8), turned to 90 degrees
- moved TP2 58.2 mm to (152.1, 117.5), turned to 90 degrees
- moved TP3 53.5 mm to (148.5, 117.5), turned to 90 degrees
- moved C5 49.3 mm to (150.5, 98.8), turned to 90 degrees
- moved C6 48.9 mm to (151.5, 98.8), turned to 90 degrees
- moved TP4 48.8 mm to (144.9, 117.5), turned to 90 degrees
- moved R4 47.0 mm to (144.2, 98.1), turned to 90 degrees
- moved R1 42.0 mm to (135.2, 92.7), turned to 90 degrees
- moved R2 39.4 mm to (137.3, 90.0)
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Connections:
- C1 pad 2: +3.3V -> GND
- C2 pad 2: unconnected-(C2-Pad2) -> GND
- C3 pad 2: unconnected-(C3-Pad2) -> GND
- C5 pad 2: +3.3V -> GND
- C6 pad 2: +3.3V -> GND
- J1 pad 1: +3.3V -> GND
- J1 pad 4: +3.3V -> /CC2
- J1 pad 5: +3.3V -> /CC1
- J1 pad 7: +3.3V -> GND
- J1 pad 8: +3.3V -> GND
- R1 pad 1: +3.3V -> /CC1
- R1 pad 2: unconnected-(R1-Pad2) -> GND
- R2 pad 1: +3.3V -> /CC2
- R2 pad 2: unconnected-(R2-Pad2) -> GND
- R3 pad 2: unconnected-(R3-Pad2) -> /EN
- R4 pad 1: +3.3V -> /SD_CTRL_A
- R4 pad 2: unconnected-(R4-Pad2) -> /SD_MODE
- SW1 pad 2: +3.3V -> GND
- SW2 pad 1: +3.3V -> /EN
- SW2 pad 2: +3.3V -> GND
- TP2 pad 1: +3.3V -> GND
- U1 pad 1: unconnected-(U1-GND-Pad1) -> GND
- U1 pad 11: unconnected-(U1-IO7-Pad11) -> /SD_CTRL_A
- U1 pad 12: unconnected-(U1-IO8-Pad12) -> /SD_CTRL_B
- U1 pad 2: unconnected-(U1-GND-Pad2) -> GND
- U1 pad 42: unconnected-(U1-GND-Pad42) -> GND
- U1 pad 43: unconnected-(U1-GND-Pad43) -> GND
- U1 pad 45: +3.3V -> /EN
- U1 pad 46: unconnected-(U1-GND-Pad46) -> GND
- U1 pad 47: unconnected-(U1-GND-Pad47) -> GND
- U1 pad 48: unconnected-(U1-GND-Pad48) -> GND
- U1 pad 49: unconnected-(U1-GND-Pad49) -> GND
- U1 pad 50: unconnected-(U1-GND-Pad50) -> GND
- U1 pad 51: unconnected-(U1-GND-Pad51) -> GND
- U1 pad 52: unconnected-(U1-GND-Pad52) -> GND
- U1 pad 53: unconnected-(U1-GND-Pad53) -> GND
- U1 pad 54: unconnected-(U1-GND-Pad54) -> GND
- U1 pad 55: unconnected-(U1-GND-Pad55) -> GND
- U1 pad 56: unconnected-(U1-GND-Pad56) -> GND
- U1 pad 57: unconnected-(U1-GND-Pad57) -> GND
- U1 pad 58: unconnected-(U1-GND-Pad58) -> GND
- U1 pad 59: unconnected-(U1-GND-Pad59) -> GND
- U1 pad 60: unconnected-(U1-GND-Pad60) -> GND
- U1 pad 61: unconnected-(U1-GND-Pad61) -> GND
- U1 pad 62: unconnected-(U1-GND-Pad62) -> GND
- U1 pad 63: unconnected-(U1-GND-Pad63) -> GND
- U1 pad 64: unconnected-(U1-GND-Pad64) -> GND
- U1 pad 65: +3.3V -> GND
- U2 pad 11: unconnected-(U2-GND-Pad11) -> GND
- U2 pad 15: unconnected-(U2-GND-Pad15) -> GND
- U2 pad 17: +3.3V -> GND
- U2 pad 3: +3.3V -> GND
- U2 pad 4: +3.3V -> /SD_MODE
- U2 pad 8: unconnected-(U2-VDD-Pad8) -> +5V
- U3 pad 1: +3.3V -> GND
- U3 pad 2: +3.3V -> GND
- U3 pad 3: +5V -> unconnected-(U3-NC-Pad3)
Routing:
- net +5V: track 0.00 -> 51.3 mm, vias 0 -> 6
- net +3.3V: track 1.10 -> 36.0 mm, vias 5 -> 4
- net /I2S_DOUT: track 0.00 -> 25.3 mm, vias 0 -> 4
- net /I2S_BCLK: track 0.00 -> 23.1 mm, vias 0 -> 4
- net /I2S_LRCLK: track 0.00 -> 18.6 mm, vias 0 -> 2
- net /SD_CTRL_A: track 0.00 -> 18.3 mm, vias 0 -> 2
- net GND: track 0.00 -> 18.2 mm, vias 0 -> 73
- net /SD_CTRL_B: track 0.00 -> 16.6 mm, vias 0 -> 2
- net /UART_TX: track 0.00 -> 16.1 mm, vias 0 -> 1
- net /USB_DP: track 0.00 -> 14.4 mm, vias 0 -> 2
- net /USB_DM: track 0.00 -> 14.4 mm, vias 0 -> 2
- net /CC2: track 0.00 -> 13.4 mm
- net /UART_RX: track 0.00 -> 9.60 mm, vias 0 -> 1
- net /SPKR_P: track 0.00 -> 9.16 mm
- net /SPKR_N: track 0.00 -> 7.55 mm
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- added copper zone on B.Cu, net GND
- added copper zone on F.Cu, net GND
- removed copper zone on B.Cu, net unconnected-(U1-GND-Pad61)
- removed copper zone on F.Cu, net unconnected-(U1-GND-Pad61)
Other:
- board size 70.5 x 41 mm -> 41 x 41 mm
